File: PCB/PCB.sch (KiCad schematic (older format))
At the start: 8 parts, among them P1 Power, P2 Analog, P3 Digital, P4 Digital, P5 CONN_01X01, P6 CONN_01X01, P7 CONN_01X01, P8 CONN_01X01

Commit message: update sch & pdf file
Parts:
- added C? (x4): 100nF, symbol C
- added C?: 100uF/6.3V, symbol CP
- added C?: 22pF, symbol C
- added C?: 1uF/6.3V, symbol CP
- added C?: 10uF/6.3V, symbol CP
- added D?: MBR0520, Diode_SMD:D_SOD-123, symbol MBR0520
- added Q?: S8550, Package_TO_SOT_THT:TO-92_Inline, symbol S8550
- added Q?: S8050, Package_TO_SOT_THT:TO-92_Inline, symbol S8050
- added R?: 21.5k, symbol R
- added R?: 10k, symbol R
- added R? (x4): R, symbol R
- added U?: LM317DCYR, symbol LM317_3PinPackage
- added U?: RT9193, symbol RT9193
- added U?: CH340C, symbol CH340C
Connections:
- net labels added: 3.3V, 3.7V, BOOT0, CHDTR, CHRTS, CHRXD, CHTXD, UD+, UD-, VUSB
- wire segments 38 -> 77
- no-connect marks 5 -> 12
Other:
- note added: "3.7V to 3.3V"
- note added: "VUSB(5V) TO 3.7V"
- moved on the sheet: P1, P2, P3, P4, P5, P6, P7, P8
