File: PCB/PCB.sch (KiCad schematic (older format))
At the start: 28 parts, among them P1 Power, P2 Analog, P3 Digital, P4 Digital, P5 CONN_01X01, P6 CONN_01X01, P7 CONN_01X01, P8 CONN_01X01

Commit message: design power
Parts:
- removed C? (x2): 100nF, symbol C
- removed C?: 100uF/6.3V, symbol CP
- removed C?: 22pF, symbol C
- removed C?: 10uF/6.3V, symbol CP
- removed D?: MBR0520, Diode_SMD:D_SOD-123, symbol MBR0520
- removed R?: 21.5k, symbol R
- removed R?: 10k, symbol R
- removed U?: LM317DCYR, symbol LM317_3PinPackage
- removed U?: RT9193, symbol RT9193
- added C? (x4): 0.1uF, symbol C
- added C? (x2): 10uF/25V, symbol CP
- added C? (x2): 10nF, symbol C
- added C?: 22uF/6.3V, symbol CP
- added C?: 100uF/6.3V, symbol CP
- added C?: 22nF, symbol C
- added C?: 10UF, symbol C
- added D?: 26V, symbol D_TVS
- added D? (x5): SS14, symbol D_Schottky
- added D?: 5V, symbol D_TVS
- added F? (x2): Polyfuse, symbol Polyfuse
- added L? (x2): 4.7uH/2.0A, symbol INDUCTOR
- added Q? (x3): AO3407, symbol Q_PMOS_GDS
- added R? (x2): 100k, symbol R
- added R? (x2): 49.9k, symbol R
- added R? (x2): 8.2k, symbol R
- added R? (x3): 10k, symbol R
- added U? (x2): MP2359, symbol MP2359
- added U?: RT9193, symbol RT9193
- added U?: STM32L151CBUx, UFQFPN48, symbol STM32L151CBUx
- C?: value 1uF/6.3V -> 10uF/6.3V
Connections:
- net labels added: +3V8, +BATT, G_EN, VBUS, VDD
- net labels removed: 3.3V, 3.7V
- wire segments 77 -> 135
Other:
- note removed: "3.7V to 3.3V"
- note removed: "VUSB(5V) TO 3.7V"
- moved on the sheet: C?, Q?, R?, U?

Commit message: pcb v0.1
Parts:
- added AE?: GPRS Antenna, symbol Antenna
- added AVDD-JP, R? (x8): 10k, symbol R
- added C? (x8): 100nF, symbol C
- added C?: 10uF, symbol C
- added C? (x2): 30pF, symbol C
- added C? (x2): 6pF, symbol C
- added D?: SS14, symbol D_Schottky
- added D?: LED, symbol LED
- added D?: LED_RGB, symbol LED_RGB
- added J?: Conn_01x03, symbol Conn_01x03
- added J?: SIM_Card, symbol SIM_Card
- added Q?: S8050, Package_TO_SOT_THT:TO-92_Inline, symbol S8050
- added R?: 1k, symbol R
- added R? (x7): 470R, symbol R
- added SW? (x4): SW_Push, symbol SW_Push
- added U?: BC95, symbol BC95
- added U?: SMF05C, symbol Conn_02x03_Counter_Clockwise
- added U?: SHT30-DIS, symbol SHT30-DIS
- added Y?: 8MHz, symbol Crystal
- added Y?: 32.768KHz, symbol Crystal
- C?: value 10UF -> 10uF
- R? (x2): value R -> 10k
- R? (x2): value R -> 1k
- U?: symbol STM32L151CBUx -> STM32L151CBUx-RESCUE-PCB
Connections:
- net labels added: BC95_RST, BC95_RXD, BC95_TXD, K1, K2, K3, LED_B, LED_G, LED_R, OSC32_IN, OSC32_OUT, SCL, SCL2, SDA, SDA2, SHT_AT, SIM_CLK, SIM_DAT, SIM_GND, SIM_RST, SIM_VDD, SWCLK, SWDIO, XI, XO
- wire segments 135 -> 265
- no-connect marks 12 -> 19
Other:
- moved on the sheet: Q?, R?, U?
